Commit message: add 2nd robot

File: gilbreth_support/urdf/gilbreth.xacro (robot description, xacro)
@@ -1,6 +1,9 @@
 <?xml version="1.0" ?>
 <robot name="gilbreth" xmlns:xacro="http://www.ros.org/wiki/xacro">
+  <!-- world -->
+  <link name="world"/>
   <!-- robot system -->
-  <xacro:include filename="$(find gilbreth_support)/urdf/robot_system/robot_system.xacro"/>
+  <xacro:include filename="$(find gilbreth_support)/urdf/robot_system/robot_system.xacro" ns="robot_system"/>
+  <xacro:include filename="$(find gilbreth_support)/urdf/robot_system/robot_place.xacro" ns="robot_place"/>
   <!-- bins -->
   <xacro:include filename="$(find gilbreth_support)/urdf/bin/bin.urdf.xacro"/>
@@ -22,4 +25,15 @@
     <parent link="world" />
     <child link="world_interface" />
+  </joint>
+  <!-- robot system link to world -->
+  <joint name="$linear_actuator_world_joint" type="fixed">
+    <parent link="world" />
+    <child link="linear_actuator_base_link" />
+    <origin xyz="0.4 0.0 0.9" rpy="0 0 0" />
+  </joint>
+  <joint name="robot_place_world_joint" type="fixed">
+    <parent link="world" />
+    <child link="robot_place_base_block" />
+    <origin xyz="0.4 0.0 0.9" rpy="0 0 0" />
   </joint>
   <!-- a break_beam type sensor in the frame break_beam_frame -->

File: gilbreth_support/urdf/linear_actuator/linear_actuator.urdf.xacro (robot description, xacro)
@@ -7,5 +7,4 @@
     <xacro:property name="carriage_length" value="0.2"/>
     <!-- link list -->
-    <link name="world"/>
     <link name="${prefix}base_link">
       <visual>
@@ -43,9 +42,4 @@
     </link>
     <!-- joint list -->
-    <joint name="${prefix}world_joint" type="fixed">
-      <parent link="world" />
-      <child link="${prefix}base_link" />
-      <origin xyz="0.4 0.0 0.9" rpy="0 0 0" />
-    </joint>
     <joint name="${prefix}carriage_joint" type="prismatic">
       <parent link="${prefix}base_link" />
